Commit message: partially fixed clipping and softened finger tips for grasping pegs

File: robotiq_s_model_visualization/cfg/robotiq_hand_macro.urdf.xacro (robot description, xacro)
@@ -12,5 +12,5 @@
     <link name="${prefix}link_0">
       <visual>
-        <origin xyz="0 0 0" rpy="0 0 0"/>
+        <origin xyz="0.02 0 0" rpy="0 0 0"/>
         <geometry>
           <mesh filename="package://robotiq_s_model_visualization/meshes/s-model_articulated/visual/link_0.STL" />
@@ -21,5 +21,5 @@
       </visual>
       <collision>
-        <origin rpy="0 0 0" xyz="0 0 0"/>
+        <origin rpy="0 3.1415926 ${-3.1415926/2}" xyz="0 0 0"/>
         <geometry>
           <mesh filename="package://robotiq_s_model_visualization/meshes/s-model_articulated/collision/link_0.STL" />
@@ -131,6 +131,8 @@
     </link>
     <gazebo reference="${prefix}link_3">
-      <mu1>1.1</mu1>
-      <mu2>1.1</mu2>
+      <mu1>1000</mu1>
+      <mu2>1000</mu2>
+      <kp>10000</kp>
+      <kd>1</kd>
     </gazebo>
     <!-- Link proximal actuating hinge -->
